Commit message: Add files via upload

File: bbr_description/urdf/bbr_robot.urdf (robot description, URDF)
Before this commit: robot bbr_robot, 11 links, 10 joints
Links:
- link IMU_link: geometry collision mesh filename=file://$(find bbr_rob)/bbr_description/meshes/IMU_link.STL; visual mesh filename=file://$(find bbr_rob)/bbr_description/meshes/IMU_link.STL
- link base_link: geometry collision mesh filename=file://$(find bbr_rob)/bbr_description/meshes/base_link.STL; visual mesh filename=file://$(find bbr_rob)/bbr_description/meshes/base_link.STL
- link camera_link: geometry collision mesh filename=file://$(find bbr_rob)/bbr_description/meshes/camera_link.S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; visual mesh filename=file://$(find bbr_rob)/bbr_description/meshes/camera_link.S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
- link front_caster_link: geometry collision mesh filename=file://$(find bbr_rob)/bbr_description/meshes/front_caster_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; visual mesh filename=file://$(find bbr_rob)/bbr_description/meshes/front_caster_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
- link left_limb_link: geometry collision mesh filename=file://$(find bbr_rob)/bbr_description/meshes/left_limb_lin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; visual mesh filename=file://$(find bbr_rob)/bbr_description/meshes/left_limb_lin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
- link left_shoulder_link: geometry collision mesh filename=file://$(find bbr_rob)/bbr_description/meshes/left_shoulder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; visual mesh filename=file://$(find bbr_rob)/bbr_description/meshes/left_shoulder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
- link left_wheel_link: geometry collision mesh filename=file://$(find bbr_rob)/bbr_description/meshes/left_wheel_li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; visual mesh filename=file://$(find bbr_rob)/bbr_description/meshes/left_wheel_li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
- link rear_caster_link: geometry collision mesh filename=file://$(find bbr_rob)/bbr_description/meshes/rear_caster_l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; visual mesh filename=file://$(find bbr_rob)/bbr_description/meshes/rear_caster_l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
- link right_limb_link: geometry collision mesh filename=file://$(find bbr_rob)/bbr_description/meshes/right_limb_li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; visual mesh filename=file://$(find bbr_rob)/bbr_description/meshes/right_limb_li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
- link right_shoulder_link: geometry collision mesh filename=file://$(find bbr_rob)/bbr_description/meshes/right_shoulde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; visual mesh filename=file://$(find bbr_rob)/bbr_description/meshes/right_shoulde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
- link right_wheel_link: geometry collision mesh filename=file://$(find bbr_rob)/bbr_description/meshes/right_wheel_l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; visual mesh filename=file://$(find bbr_rob)/bbr_description/meshes/right_wheel_l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
